Commit message: edit sensor positions

File: husky_description/urdf/husky_macro.urdf.xacro (robot description, xacro)
@@ -112,5 +112,5 @@
       <parent link="top_plate_link" />
       <child link="lidar_link"/>
-      <origin xyz="0.2206 0.0 0.008" rpy="0 0 0" />
+      <origin xyz="0 0.0 0.0275" rpy="0 0 0" />
       <!--
       <parent link="base_link"/>
@@ -140,7 +140,7 @@
     </link>
     <joint name="camera_joint" type="fixed">
-      <parent link="base_link"/>
+      <parent link="top_plate_link"/>
       <child link="camera_link"/>
-      <origin xyz="0.4 0 0.15" rpy="0 0 0"/>
+      <origin xyz="0.353 0.0 -0.01" rpy="0 0 0"/>
     </joint>
     <link name="camera_depth_frame"/>
